File: raspberrypi-gpio-40pin.kicad_pcb (KiCad board)
At the start: 2 copper layers, 65 x 56 mm, 15 parts, among them J1 Conn_01x02_Female, J10 Conn_01x02_Female, J2 Conn_01x02_Female, J3 Conn_01x02_Female, J4 Conn_01x02_Female, J5 Conn_01x02_Female, J6 Conn_01x02_Female, J7 Conn_01x02_Female, J8 Conn_01x02_Female, J9 Conn_01x02_Female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

Commit message: mika
Parts:
- moved TR2 7.45 mm to (203.3, 97.5)
Routing:
- net +5V: track 18.9 -> 34.6 mm
- added copper zone on F.Cu, net (none)
- added copper zone on F.Cu, net +5V
Other:
- outline, holes or cut-outs redrawn
