File: raspberrypi-gpio-40pin.kicad_pcb (KiCad board)
At the start: 2 copper layers, 65 x 56 mm, 35 parts, among them J1 Conn_01x02_Female, J10 Conn_01x02_Female, J11 Conn_01x02_Male, J12 Conn_01x02_Male, J13 Conn_01x02_Male, J14 Conn_01x02_Male, J15 Conn_01x02_Male, J16 Conn_01x02_Male, J17 Conn_01x02_Male, J18 Conn_01x02_Male, J19 Conn_01x02_Male, J2 Conn_01x02_Female, J20 Conn_01x02_Male, J21 Conn_01x02_Male, J22 Conn_01x02_Male, J23 Conn_01x02_Male, J24 Conn_01x02_Male, J25 Conn_01x02_Male, J26 Conn_01x02_Male, J27 Conn_01x02_Male, J28 Conn_01x02_Male, J29 Conn_01x02_Male, J3 Conn_01x02_Female, J30 Conn_01x02_Male, J4 Conn_01x02_Female, J5 Conn_01x02_Female, J6 Conn_01x02_Female, J7 Conn_01x02_Female, J8 Conn_01x02_Female, J9 Conn_01x02_Female, P1 Conn_02x20_Odd_Even

Commit message: tt
Routing:
- net GND: track 419.7 -> 878.0 mm
- net +3V3: track 62.8 -> 125.7 mm
- net +5V: track 57.9 -> 115.7 mm
- net /GPIO5: track 51.7 -> 103.3 mm
- net /GPIO22(GEN3): track 51.1 -> 102.2 mm
- net /GPIO26: track 49.3 -> 98.6 mm
- net /GPIO27(GEN2): track 48.0 -> 96.0 mm
- net /GPIO4(GCLK): track 46.9 -> 93.9 mm
- net /GPIO17(GEN0): track 44.6 -> 89.2 mm
- net /GPIO13(PWM1): track 42.2 -> 84.4 mm
- net /GPIO6: track 42.0 -> 84.0 mm
- added copper zone on B.Cu, net (none)
- added copper zone on B.Cu, net +3V3
- added copper zone on B.Cu, net +5V
- added copper zone on B.Cu, net /GPIO26
- added copper zone on B.Cu, net GND

Commit message: ghgf
Routing:
- net GND: track 878.0 -> 839.4 mm
Changed lines of the file:
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@@
     (thickness 1.6)
     (drawings 59)
-    (tracks 501)
+    (tracks 496)
     (zones 0)
     (modules 35)
@@
   (segment (start 209.5 145) (end 212 147.5) (width 1) (layer F.Cu) (net 3))
   (segment (start 209.5 142.25) (end 209.5 145) (width 1) (layer F.Cu) (net 3))
-  (segment (start 238.85 123.649776) (end 247.800224 132.6) (width 1) (layer F.Cu) (net 3))
-  (segment (start 238.85 98.77) (end 238.85 123.649776) (width 1) (layer F.Cu) (net 3))
-  (segment (start 247.800224 132.6) (end 248.9 132.6) (width 1) (layer F.Cu) (net 3))
   (segment (start 254.5 142.25) (end 254.5 139.775127) (width 1) (layer B.Cu) (net 6))
   (segment (start 251.44 132.6) (end 251.44 136.3) (width 1) (layer B.Cu) (net 6))
@@
   (segment (start 254.5 142.25) (end 254.5 139.775127) (width 1) (layer F.Cu) (net 6))
   (segment (start 251.44 132.6) (end 251.44 130.5) (width 1) (layer F.Cu) (net 6))
+  (segment (start 251.44 130.5) (end 250.84001 129.90001) (width 1) (layer F.Cu) (net 6))
+  (segment (start 250.84001 129.90001) (end 247.221569 129.90001) (width 1) (layer F.Cu) (net 6))
+  (segment (start 247.221569 129.90001) (end 243.390001 126.068442) (width 1) (layer F.Cu) (net 6))
+  (segment (start 243.390001 126.068442) (end 243.390001 100.724212) (width 1) (layer F.Cu) (net 6))
   (segment (start 243.390001 100.724212) (end 243.93 100.184213) (width 1) (layer F.Cu) (net 6))
-  (segment (start 243.500009 126.17845) (end 243.500009 125.978675) (width 1) (layer F.Cu) (net 6))
   (segment (start 243.93 100.184213) (end 243.93 98.77) (width 1) (layer F.Cu) (net 6))
-  (segment (start 243.390001 125.868667) (end 243.390001 100.724212) (width 1) (layer F.Cu) (net 6))
-  (segment (start 250.84001 129.90001) (end 247.221569 129.90001) (width 1) (layer F.Cu) (net 6))
-  (segment (start 251.44 130.5) (end 250.84001 129.90001) (width 1) (layer F.Cu) (net 6))
-  (segment (start 243.500009 125.978675) (end 243.390001 125.868667) (width 1) (layer F.Cu) (net 6))
-  (segment (start 247.221569 129.90001) (end 243.500009 126.17845) (width 1) (layer F.Cu) (net 6))
   (segment (start 258.25 127.75) (end 257.4 126.9) (width 1) (layer B.Cu) (net 7))
   (segment (start 246.2 125.36) (end 248.3 125.36) (width 1) (layer B.Cu) (net 7))
@@
   (segment (start 244.5 142.25) (end 244.5 137.3) (width 1) (layer F.Cu) (net 16))
   (segment (start 244.5 137.3) (end 243.2 136) (width 1) (layer F.Cu) (net 16))
-  (segment (start 235.100011 108.558678) (end 226.15 99.608668) (width 1) (layer F.Cu) (net 16))
-  (segment (start 243.2 132.4) (end 243.2 130.12111) (width 1) (layer F.Cu) (net 16))
-  (segment (start 235.100011 122.021122) (end 235.100011 108.558678) (width 1) (layer F.Cu) (net 16))
-  (segment (start 243.2 130.12111) (end 235.100011 122.021122) (width 1) (layer F.Cu) (net 16))
-  (segment (start 226.15 99.608668) (end 226.15 98.77) (width 1) (layer F.Cu) (net 16))
   (segment (start 226.15 99.608668) (end 226.15 98.77) (width 1) (layer B.Cu) (net 16))
   (segment (start 235.100011 108.558678) (end 226.15 99.608668) (width 1) (layer B.Cu) (net 16))
@@
   (segment (start 243.2 132.4) (end 243.2 127.999775) (width 1) (layer B.Cu) (net 16))
   (segment (start 243.2 127.999775) (end 235.100011 119.899786) (width 1) (layer B.Cu) (net 16))
+  (segment (start 243.2 132.4) (end 243.2 127.999775) (width 1) (layer F.Cu) (net 16))
+  (segment (start 226.15 99.608668) (end 226.15 98.77) (width 1) (layer F.Cu) (net 16))
+  (segment (start 235.100011 108.558678) (end 226.15 99.608668) (width 1) (layer F.Cu) (net 16))
+  (segment (start 235.100011 119.899786) (end 235.100011 108.558678) (width 1) (layer F.Cu) (net 16))
+  (segment (start 243.2 127.999775) (end 235.100011 119.899786) (width 1) (layer F.Cu) (net 16))
   (segment (start 253.05 117.75) (end 252.1 118.7) (width 1) (layer B.Cu) (net 26))
   (segment (start 258.25 117.75) (end 253.05 117.75) (width 1) (layer B.Cu) (net 26))

Commit message: ffhg
Routing:
- net GND: track 839.4 -> 891.7 mm
Other:
- net class Default: clearance 0.5 -> 0.8
- rule trace_clearance: 0.5 -> 0.8
Changed lines of the file:
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@@
     (thickness 1.6)
     (drawings 59)
-    (tracks 496)
+    (tracks 503)
     (zones 0)
     (modules 35)
@@
     (0 F.Cu signal)
     (31 B.Cu signal)
-    (32 B.Adhes user hide)
-    (33 F.Adhes user hide)
-    (34 B.Paste user hide)
-    (35 F.Paste user hide)
-    (36 B.SilkS user hide)
+    (32 B.Adhes user)
+    (33 F.Adhes user)
+    (34 B.Paste user)
+    (35 F.Paste user)
+    (36 B.SilkS user)
     (37 F.SilkS user)
-    (38 B.Mask user hide)
-    (39 F.Mask user hide)
-    (40 Dwgs.User user hide)
-    (41 Cmts.User user hide)
-    (42 Eco1.User user hide)
-    (43 Eco2.User user hide)
-    (44 Edge.Cuts user hide)
-    (45 Margin user hide)
-    (46 B.CrtYd user hide)
-    (47 F.CrtYd user hide)
+    (38 B.Mask user)
+    (39 F.Mask user)
+    (40 Dwgs.User user)
+    (41 Cmts.User user)
+    (42 Eco1.User user)
+    (43 Eco2.User user)
+    (44 Edge.Cuts user)
+    (45 Margin user)
+    (46 B.CrtYd user)
+    (47 F.CrtYd user)
   )
   (setup
     (last_trace_width 1)
-    (trace_clearance 0.5)
+    (trace_clearance 0.8)
     (zone_clearance 0.508)
     (zone_45_only no)
@@
   (net 31 "Net-(P1-Pad19)")
   (net_class Default "This is the default net class."
-    (clearance 0.5)
+    (clearance 0.8)
     (trace_width 1)
     (via_dia 0.9)
@@
   (segment (start 209.5 145) (end 212 147.5) (width 1) (layer F.Cu) (net 3))
   (segment (start 209.5 142.25) (end 209.5 145) (width 1) (layer F.Cu) (net 3))
+  (segment (start 238.85 98.77) (end 238.85 123.649776) (width 1) (layer F.Cu) (net 3))
+  (segment (start 238.85 123.649776) (end 247.800224 132.6) (width 1) (layer F.Cu) (net 3))
+  (segment (start 247.800224 132.6) (end 248.9 132.6) (width 1) (layer F.Cu) (net 3))
+  (segment (start 248.9 132.6) (end 247.800224 132.6) (width 1) (layer B.Cu) (net 3))
+  (segment (start 247.800224 132.6) (end 238.9 123.699776) (width 1) (layer B.Cu) (net 3))
   (segment (start 254.5 142.25) (end 254.5 139.775127) (width 1) (layer B.Cu) (net 6))
   (segment (start 251.44 132.6) (end 251.44 136.3) (width 1) (layer B.Cu) (net 6))
@@
   (segment (start 254.5 142.25) (end 254.5 139.775127) (width 1) (layer F.Cu) (net 6))
   (segment (start 251.44 132.6) (end 251.44 130.5) (width 1) (layer F.Cu) (net 6))
+  (segment (start 243.390001 100.724212) (end 243.93 100.184213) (width 1) (layer F.Cu) (net 6))
+  (segment (start 243.500009 126.17845) (end 243.500009 125.978675) (width 1) (layer F.Cu) (net 6))
+  (segment (start 243.93 100.184213) (end 243.93 98.77) (width 1) (layer F.Cu) (net 6))
+  (segment (start 243.390001 125.868667) (end 243.390001 100.724212) (width 1) (layer F.Cu) (net 6))
+  (segment (start 250.84001 129.90001) (end 247.221569 129.90001) (width 1) (layer F.Cu) (net 6))
   (segment (start 251.44 130.5) (end 250.84001 129.90001) (width 1) (layer F.Cu) (net 6))
-  (segment (start 250.84001 129.90001) (end 247.221569 129.90001) (width 1) (layer F.Cu) (net 6))
-  (segment (start 247.221569 129.90001) (end 243.390001 126.068442) (width 1) (layer F.Cu) (net 6))
-  (segment (start 243.390001 126.068442) (end 243.390001 100.724212) (width 1) (layer F.Cu) (net 6))
-  (segment (start 243.390001 100.724212) (end 243.93 100.184213) (width 1) (layer F.Cu) (net 6))
-  (segment (start 243.93 100.184213) (end 243.93 98.77) (width 1) (layer F.Cu) (net 6))
+  (segment (start 243.500009 125.978675) (end 243.390001 125.868667) (width 1) (layer F.Cu) (net 6))
+  (segment (start 247.221569 129.90001) (end 243.500009 126.17845) (width 1) (layer F.Cu) (net 6))
   (segment (start 258.25 127.75) (end 257.4 126.9) (width 1) (layer B.Cu) (net 7))
   (segment (start 246.2 125.36) (end 248.3 125.36) (width 1) (layer B.Cu) (net 7))
@@
   (segment (start 244.5 142.25) (end 244.5 137.3) (width 1) (layer F.Cu) (net 16))
   (segment (start 244.5 137.3) (end 243.2 136) (width 1) (layer F.Cu) (net 16))
+  (segment (start 235.100011 108.558678) (end 226.15 99.608668) (width 1) (layer F.Cu) (net 16))
+  (segment (start 243.2 132.4) (end 243.2 130.12111) (width 1) (layer F.Cu) (net 16))
+  (segment (start 235.100011 122.021122) (end 235.100011 108.558678) (width 1) (layer F.Cu) (net 16))
+  (segment (start 243.2 130.12111) (end 235.100011 122.021122) (width 1) (layer F.Cu) (net 16))
+  (segment (start 226.15 99.608668) (end 226.15 98.77) (width 1) (layer F.Cu) (net 16))
+  (segment (start 235.100011 122.021122) (end 235.100011 108.558678) (width 1) (layer B.Cu) (net 16))
+  (segment (start 235.100011 108.558678) (end 226.15 99.608668) (width 1) (layer B.Cu) (net 16))
+  (segment (start 243.2 130.12111) (end 235.100011 122.021122) (width 1) (layer B.Cu) (net 16))
+  (segment (start 243.2 132.4) (end 243.2 130.12111) (width 1) (layer B.Cu) (net 16))
   (segment (start 226.15 99.608668) (end 226.15 98.77) (width 1) (layer B.Cu) (net 16))
-  (segment (start 235.100011 108.558678) (end 226.15 99.608668) (width 1) (layer B.Cu) (net 16))
-  (segment (start 235.100011 119.899786) (end 235.100011 108.558678) (width 1) (layer B.Cu) (net 16))
-  (segment (start 243.2 132.4) (end 243.2 127.999775) (width 1) (layer B.Cu) (net 16))
-  (segment (start 243.2 127.999775) (end 235.100011 119.899786) (width 1) (layer B.Cu) (net 16))
-  (segment (start 243.2 132.4) (end 243.2 127.999775) (width 1) (layer F.Cu) (net 16))
-  (segment (start 226.15 99.608668) (end 226.15 98.77) (width 1) (layer F.Cu) (net 16))
-  (segment (start 235.100011 108.558678) (end 226.15 99.608668) (width 1) (layer F.Cu) (net 16))
-  (segment (start 235.100011 119.899786) (end 235.100011 108.558678) (width 1) (layer F.Cu) (net 16))
-  (segment (start 243.2 127.999775) (end 235.100011 119.899786) (width 1) (layer F.Cu) (net 16))
   (segment (start 253.05 117.75) (end 252.1 118.7) (width 1) (layer B.Cu) (net 26))
   (segment (start 258.25 117.75) (end 253.05 117.75) (width 1) (layer B.Cu) (net 26))

Commit message: dcsd
Routing:
- net /GPIO5: track 103.3 -> 72.5 mm
- net GND: track 891.7 -> 916.6 mm
Changed lines of the file:
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@@
     (thickness 1.6)
     (drawings 59)
-    (tracks 503)
+    (tracks 500)
     (zones 0)
     (modules 35)
@@
   (segment (start 211 109.974873) (end 211 106) (width 1) (layer F.Cu) (net 2))
   (segment (start 208.37 96.23) (end 210.91 96.23) (width 1) (layer F.Cu) (net 2))
+  (segment (start 238.85 98.77) (end 238.85 123.649776) (width 1) (layer B.Cu) (net 3))
   (segment (start 209.5 142.25) (end 209.5 145) (width 1) (layer B.Cu) (net 3))
   (segment (start 209.5 145) (end 212 147.5) (width 1) (layer B.Cu) (net 3))
@@
   (segment (start 209.5 145) (end 212 147.5) (width 1) (layer F.Cu) (net 3))
   (segment (start 209.5 142.25) (end 209.5 145) (width 1) (layer F.Cu) (net 3))
-  (segment (start 238.85 98.77) (end 238.85 123.649776) (width 1) (layer F.Cu) (net 3))
   (segment (start 238.85 123.649776) (end 247.800224 132.6) (width 1) (layer F.Cu) (net 3))
   (segment (start 247.800224 132.6) (end 248.9 132.6) (width 1) (layer F.Cu) (net 3))
   (segment (start 248.9 132.6) (end 247.800224 132.6) (width 1) (layer B.Cu) (net 3))
   (segment (start 247.800224 132.6) (end 238.9 123.699776) (width 1) (layer B.Cu) (net 3))
+  (segment (start 238.85 98.77) (end 238.85 123.649776) (width 1) (layer F.Cu) (net 3))
   (segment (start 254.5 142.25) (end 254.5 139.775127) (width 1) (layer B.Cu) (net 6))
   (segment (start 251.44 132.6) (end 251.44 136.3) (width 1) (layer B.Cu) (net 6))
@@
   (segment (start 251.44 132.6) (end 251.44 130.5) (width 1) (layer F.Cu) (net 6))
   (segment (start 243.390001 100.724212) (end 243.93 100.184213) (width 1) (layer F.Cu) (net 6))
-  (segment (start 243.500009 126.17845) (end 243.500009 125.978675) (width 1) (layer F.Cu) (net 6))
   (segment (start 243.93 100.184213) (end 243.93 98.77) (width 1) (layer F.Cu) (net 6))
-  (segment (start 243.390001 125.868667) (end 243.390001 100.724212) (width 1) (layer F.Cu) (net 6))
   (segment (start 250.84001 129.90001) (end 247.221569 129.90001) (width 1) (layer F.Cu) (net 6))
   (segment (start 251.44 130.5) (end 250.84001 129.90001) (width 1) (layer F.Cu) (net 6))
-  (segment (start 243.500009 125.978675) (end 243.390001 125.868667) (width 1) (layer F.Cu) (net 6))
-  (segment (start 247.221569 129.90001) (end 243.500009 126.17845) (width 1) (layer F.Cu) (net 6))
   (segment (start 258.25 127.75) (end 257.4 126.9) (width 1) (layer B.Cu) (net 7))
   (segment (start 246.2 125.36) (end 248.3 125.36) (width 1) (layer B.Cu) (net 7))

Commit message: logo
Parts:
- added G***: LOGO, atx:logo3, F.Cu at (239.4, 120.2)
- added G***: LOGO, atx:logo3, F.Cu at (219.8, 120.5)
Routing:
- net /GPIO5: track 72.5 -> 103.3 mm
Other:
- board text added: "gpio13 -"
- board text added: "gpio17 -"
- board text added: "gpio22 -"
- board text added: "gpio27 -"
- board text added: "gpio4 -"
- board text added: "gpio5 -"
- board text added: "gpio6 -"
- board text added: "les raspberrys sont de la merdes heureusement arduino est mon sauveur"
