File: raspberrypi-gpio-40pin.kicad_pcb (KiCad board)
At the start: 2 copper layers, 65 x 56 mm, 37 parts, among them J1 Conn_01x02_Female, J10 Conn_01x02_Female, J11 Conn_01x02_Male, J12 Conn_01x02_Male, J13 Conn_01x02_Male, J14 Conn_01x02_Male, J15 Conn_01x02_Male, J16 Conn_01x02_Male, J17 Conn_01x02_Male, J18 Conn_01x02_Male, J19 Conn_01x02_Male, J2 Conn_01x02_Female, J20 Conn_01x02_Male, J21 Conn_01x02_Male, J22 Conn_01x02_Male, J23 Conn_01x02_Male, J24 Conn_01x02_Male, J25 Conn_01x02_Male, J26 Conn_01x02_Male, J27 Conn_01x02_Male, J28 Conn_01x02_Male, J29 Conn_01x02_Male, J3 Conn_01x02_Female, J30 Conn_01x02_Male, J4 Conn_01x02_Female, J5 Conn_01x02_Female, J6 Conn_01x02_Female, J7 Conn_01x02_Female, J8 Conn_01x02_Female, J9 Conn_01x02_Female, P1 Conn_02x20_Odd_Even

Commit message: utfuft
Parts:
- removed the G*** at (239.4, 120.2)
Changed lines of the file:
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@@
     (tracks 502)
     (zones 0)
-    (modules 37)
+    (modules 36)
     (nets 32)
   )
@@
   )
   (module atx:logo3 (layer F.Cu)
-    (at 239.4 120.2)
-    (fp_text reference G*** (at 0 0) (layer F.SilkS) hide
-      (effects (font (size 1.524 1.524) (thickness 0.3)))
-    )
-    (fp_text value LOGO (at 0.75 0) (layer F.SilkS) hide
-      (effects (font (size 1.524 1.524) (thickness 0.3)))
-    )
-    (fp_poly (pts (xy 1.337353 -1.005917) (xy 1.527379 -0.941065) (xy 1.677048 -0.830202) (xy 1.784739 -0.685245)
-      (xy 1.848831 -0.518106) (xy 1.867704 -0.340703) (xy 1.839736 -0.164949) (xy 1.763306 -0.002761)
-      (xy 1.636794 0.133948) (xy 1.5034 0.214731) (xy 1.315907 0.269455) (xy 1.124015 0.272916)
-      (xy 0.970139 0.231646) (xy 0.90204 0.187029) (xy 0.800869 0.10388) (xy 0.681748 -0.004803)
-      (xy 0.589286 -0.095699) (xy 0.330636 -0.358593) (xy 0.776111 -0.358593) (xy 0.805823 -0.270449)
-      (xy 0.891851 -0.221205) (xy 0.977194 -0.211667) (xy 1.057069 -0.204729) (xy 1.088577 -0.171018)
-      (xy 1.093611 -0.108354) (xy 1.111963 -0.013373) (xy 1.149047 0.050396) (xy 1.201678 0.096074)
-      (xy 1.24669 0.098497) (xy 1.307597 0.069314) (xy 1.361468 0.007293) (xy 1.375833 -0.089436)
-      (xy 1.382123 -0.172004) (xy 1.412461 -0.205639) (xy 1.474611 -0.211667) (xy 1.58518 -0.23581)
-      (xy 1.647687 -0.303001) (xy 1.658055 -0.358593) (xy 1.626507 -0.426483) (xy 1.546571 -0.476292)
-      (xy 1.448708 -0.493889) (xy 1.391228 -0.514192) (xy 1.375833 -0.579198) (xy 1.36018 -0.69989)
-      (xy 1.310569 -0.762928) (xy 1.249828 -0.776111) (xy 1.165092 -0.744572) (xy 1.109225 -0.660982)
-      (xy 1.093611 -0.566764) (xy 1.074641 -0.510472) (xy 1.006959 -0.493909) (xy 1.003097 -0.493889)
-      (xy 0.887354 -0.474869) (xy 0.805595 -0.425099) (xy 0.776111 -0.358593) (xy 0.330636 -0.358593)
-      (xy 0.314268 -0.375229) (xy 0.612626 -0.661665) (xy 0.792336 -0.823352) (xy 0.944094 -0.932626)
-      (xy 1.079934 -0.995204) (xy 1.211893 -1.016803) (xy 1.337353 -1.005917)) (layer Eco2.User) (width 0.01))
-    (fp_poly (pts (xy -1.246311 -0.983454) (xy -1.10286 -0.917167) (xy -0.943586 -0.801166) (xy -0.787245 -0.659965)
-      (xy -0.490657 -0.375229) (xy -0.765676 -0.096856) (xy -0.88733 0.022176) (xy -1.00084 0.125972)
-      (xy -1.091525 0.201497) (xy -1.135957 0.231869) (xy -1.25626 0.26816) (xy -1.410393 0.278993)
-      (xy -1.566375 0.264347) (xy -1.675695 0.232221) (xy -1.843572 0.124146) (xy -1.96017 -0.018966)
-      (xy -2.026874 -0.185203) (xy -2.045071 -0.362652) (xy -2.044095 -0.368617) (xy -1.799167 -0.368617)
-      (xy -1.77611 -0.308218) (xy -1.743731 -0.267104) (xy -1.679923 -0.239258) (xy -1.56641 -0.220247)
-      (xy -1.423516 -0.210316) (xy -1.271567 -0.209712) (xy -1.130889 -0.218684) (xy -1.021807 -0.237477)
-      (xy -0.973532 -0.257741) (xy -0.925115 -0.333036) (xy -0.922692 -0.390032) (xy -0.930755 -0.427963)
-      (xy -0.950648 -0.453145) (xy -0.995129 -0.468688) (xy -1.076955 -0.4777) (xy -1.20888 -0.483288)
-      (xy -1.317819 -0.486301) (xy -1.517046 -0.487834) (xy -1.655504 -0.478704) (xy -1.742479 -0.456641)
-      (xy -1.787256 -0.419375) (xy -1.799167 -0.368617) (xy -2.044095 -0.368617) (xy -2.016147 -0.539399)
-      (xy -1.941487 -0.703531) (xy -1.822478 -0.843136) (xy -1.660506 -0.946299) (xy -1.533729 -0.987971)
-      (xy -1.385935 -1.005298) (xy -1.246311 -0.983454)) (layer Eco2.User) (width 0.01))
-    (fp_poly (pts (xy 0.158733 -3.590057) (xy 0.355664 -3.577436) (xy 0.436411 -3.566439) (xy 0.862729 -3.457236)
-      (xy 1.269212 -3.284931) (xy 1.649045 -3.055765) (xy 1.99541 -2.775981) (xy 2.301492 -2.45182)
-      (xy 2.560474 -2.089525) (xy 2.765539 -1.695338) (xy 2.900729 -1.309849) (xy 2.940528 -1.110286)
-      (xy 2.967318 -0.864144) (xy 2.980915 -0.591853) (xy 2.981139 -0.313839) (xy 2.967808 -0.050532)
-      (xy 2.940739 0.177641) (xy 2.915049 0.299861) (xy 2.769094 0.722806) (xy 2.564104 1.113563)
-      (xy 2.296621 1.47787) (xy 2.041142 1.748539) (xy 1.734927 2.015845) (xy 1.427769 2.226282)
-      (xy 1.100867 2.39124) (xy 0.79375 2.504102) (xy 0.673142 2.537762) (xy 0.547213 2.561735)
-      (xy 0.398856 2.578013) (xy 0.210963 2.588582) (xy 0.017639 2.594333) (xy -0.185117 2.596538)
-      (xy -0.378105 2.594334) (xy -0.543095 2.588225) (xy -0.661858 2.578713) (xy -0.687917 2.574892)
-      (xy -1.078147 2.473705) (xy -1.466172 2.313218) (xy -1.831677 2.102321) (xy -1.937108 2.028192)
-      (xy -2.298192 1.720713) (xy -2.604449 1.372435) (xy -2.852752 0.988038) (xy -3.039973 0.572199)
-      (xy -3.142674 0.224363) (xy -3.183907 -0.023873) (xy -3.205192 -0.309665) (xy -3.205683 -0.389739)
-      (xy -2.624801 -0.389739) (xy -2.607612 -0.12355) (xy -2.54588 0.10177) (xy -2.432725 0.305012)
-      (xy -2.319782 0.443613) (xy -2.09254 0.644491) (xy -1.839492 0.781823) (xy -1.567336 0.853885)
-      (xy -1.282771 0.858951) (xy -0.992496 0.795299) (xy -0.975894 0.789557) (xy -0.795704 0.699984)
-      (xy -0.593154 0.55266) (xy -0.376145 0.353568) (xy -0.309412 0.284649) (xy -0.213567 0.186451)
-      (xy -0.13489 0.111971) (xy -0.086441 0.073356) (xy -0.079279 0.070555) (xy -0.044733 0.094241)
-      (xy 0.027816 0.158541) (xy 0.127358 0.253314) (xy 0.230133 0.355482) (xy 0.417263 0.534896)
-      (xy 0.579942 0.664274) (xy 0.733756 0.75168) (xy 0.89429 0.805177) (xy 1.07713 0.832825)
-      (xy 1.164166 0.838661) (xy 1.335805 0.842823) (xy 1.465915 0.833128) (xy 1.582753 0.806132)
-      (xy 1.665168 0.777599) (xy 1.900955 0.653153) (xy 2.111106 0.472723) (xy 2.280877 0.250032)
-      (xy 2.331777 0.157101) (xy 2.392217 0.02351) (xy 2.426044 -0.089567) (xy 2.440488 -0.214672)
-      (xy 2.442947 -0.343308) (xy 2.420372 -0.624237) (xy 2.349067 -0.864412) (xy 2.222783 -1.079412)
-      (xy 2.084211 -1.237545) (xy 1.88185 -1.409299) (xy 1.673193 -1.519202) (xy 1.441483 -1.573603)
-      (xy 1.181805 -1.579505) (xy 0.989639 -1.561232) (xy 0.826541 -1.523427) (xy 0.677077 -1.458204)
-      (xy 0.525809 -1.357676) (xy 0.3573 -1.213957) (xy 0.231676 -1.094098) (xy -0.091149 -0.777515)
-      (xy -0.385348 -1.073251) (xy -0.579553 -1.258551) (xy -0.74806 -1.393179) (xy -0.905511 -1.484347)
-      (xy -1.066548 -1.539267) (xy -1.245813 -1.565152) (xy -1.393473 -1.569861) (xy -1.562321 -1.566537)
-      (xy -1.686564 -1.553444) (xy -1.791969 -1.525901) (xy -1.904303 -1.479225) (xy -1.911932 -1.475663)
-      (xy -2.137683 -1.335986) (xy -2.337942 -1.147415) (xy -2.493374 -0.929326) (xy -2.531031 -0.855282)
-      (xy -2.586292 -0.712482) (xy -2.61521 -0.570103) (xy -2.624762 -0.393511) (xy -2.624801 -0.389739)
-      (xy -3.205683 -0.389739) (xy -3.207046 -0.611655) (xy -3.189982 -0.908483) (xy -3.154517 -1.178791)
-      (xy -3.103649 -1.393473) (xy -2.936259 -1.810866) (xy -2.707852 -2.208281) (xy -2.427665 -2.572266)
-      (xy -2.104934 -2.889372) (xy -2.039264 -2.943455) (xy -1.816892 -3.10016) (xy -1.554754 -3.251683)
-      (xy -1.279405 -3.384415) (xy -1.017398 -3.484749) (xy -0.934861 -3.509395) (xy -0.7721 -3.541764)
-      (xy -0.560215 -3.566894) (xy -0.320351 -3.583906) (xy -0.073654 -3.59192) (xy 0.158733 -3.590057)) (layer Eco2.User) (width 0.01))
-  )
-  (module atx:logo3 (layer F.Cu)

Commit message: ytfyf
Parts:
- moved G*** 19.6 mm to (239.4, 120.2)
Changed lines of the file:
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@@
   )
   (module atx:logo3 (layer F.Cu)
-    (at 219.8 120.5)
+    (at 239.4 120.2)
     (fp_text reference G*** (at 0 0) (layer F.SilkS) hide
       (effects (font (size 1.524 1.524) (thickness 0.3)))
@@
       (xy 0.887354 -0.474869) (xy 0.805595 -0.425099) (xy 0.776111 -0.358593) (xy 0.330636 -0.358593)
       (xy 0.314268 -0.375229) (xy 0.612626 -0.661665) (xy 0.792336 -0.823352) (xy 0.944094 -0.932626)
-      (xy 1.079934 -0.995204) (xy 1.211893 -1.016803) (xy 1.337353 -1.005917)) (layer Eco2.User) (width 0.01))
+      (xy 1.079934 -0.995204) (xy 1.211893 -1.016803) (xy 1.337353 -1.005917)) (layer F.SilkS) (width 0.01))
     (fp_poly (pts (xy -1.246311 -0.983454) (xy -1.10286 -0.917167) (xy -0.943586 -0.801166) (xy -0.787245 -0.659965)
       (xy -0.490657 -0.375229) (xy -0.765676 -0.096856) (xy -0.88733 0.022176) (xy -1.00084 0.125972)
@@
       (xy -1.787256 -0.419375) (xy -1.799167 -0.368617) (xy -2.044095 -0.368617) (xy -2.016147 -0.539399)
       (xy -1.941487 -0.703531) (xy -1.822478 -0.843136) (xy -1.660506 -0.946299) (xy -1.533729 -0.987971)
-      (xy -1.385935 -1.005298) (xy -1.246311 -0.983454)) (layer Eco2.User) (width 0.01))
+      (xy -1.385935 -1.005298) (xy -1.246311 -0.983454)) (layer F.SilkS) (width 0.01))
     (fp_poly (pts (xy 0.158733 -3.590057) (xy 0.355664 -3.577436) (xy 0.436411 -3.566439) (xy 0.862729 -3.457236)
       (xy 1.269212 -3.284931) (xy 1.649045 -3.055765) (xy 1.99541 -2.775981) (xy 2.301492 -2.45182)
@@
       (xy -2.104934 -2.889372) (xy -2.039264 -2.943455) (xy -1.816892 -3.10016) (xy -1.554754 -3.251683)
       (xy -1.279405 -3.384415) (xy -1.017398 -3.484749) (xy -0.934861 -3.509395) (xy -0.7721 -3.541764)
-      (xy -0.560215 -3.566894) (xy -0.320351 -3.583906) (xy -0.073654 -3.59192) (xy 0.158733 -3.590057)) (layer Eco2.User) (width 0.01))
+      (xy -0.560215 -3.566894) (xy -0.320351 -3.583906) (xy -0.073654 -3.59192) (xy 0.158733 -3.590057)) (layer F.SilkS) (width 0.01))
   )
   (module atx:PinHeader_1x02_P2.54mm_Vertical (layer F.Cu)
@@
       (net 3 GND))
   )
+  (gr_text gpio22 (at 244.3 148.1) (layer F.SilkS)
+    (effects (font (size 1 1) (thickness 0.15)))
+  )
   (gr_text "les raspberrys sont de la merdes\nheureusement\narduino est mon sauveur" (at 228.3 107.8) (layer F.SilkS)
     (effects (font (size 1 1) (thickness 0.15)))
@@
     (effects (font (size 1 1) (thickness 0.15)))
   )
-  (gr_text gpio22 (at 244.3 148.1) (layer F.SilkS)
-    (effects (font (size 1 1) (thickness 0.15)))
-  )

Commit message: quasi final
Parts:
- added G***: LOGO, atx:logo3, F.Cu at (219.8, 120.5)
Changed lines of the file:
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@@
     (tracks 502)
     (zones 0)
-    (modules 36)
+    (modules 37)
     (nets 32)
   )
@@
   )
   (module atx:logo3 (layer F.Cu)
+    (at 219.8 120.5)
+    (fp_text reference G*** (at 0 0) (layer B.SilkS) hide
+      (effects (font (size 1.524 1.524) (thickness 0.3)))
+    )
+    (fp_text value LOGO (at 0.75 0) (layer B.SilkS) hide
+      (effects (font (size 1.524 1.524) (thickness 0.3)))
+    )
+    (fp_poly (pts (xy 1.337353 -1.005917) (xy 1.527379 -0.941065) (xy 1.677048 -0.830202) (xy 1.784739 -0.685245)
+      (xy 1.848831 -0.518106) (xy 1.867704 -0.340703) (xy 1.839736 -0.164949) (xy 1.763306 -0.002761)
+      (xy 1.636794 0.133948) (xy 1.5034 0.214731) (xy 1.315907 0.269455) (xy 1.124015 0.272916)
+      (xy 0.970139 0.231646) (xy 0.90204 0.187029) (xy 0.800869 0.10388) (xy 0.681748 -0.004803)
+      (xy 0.589286 -0.095699) (xy 0.330636 -0.358593) (xy 0.776111 -0.358593) (xy 0.805823 -0.270449)
+      (xy 0.891851 -0.221205) (xy 0.977194 -0.211667) (xy 1.057069 -0.204729) (xy 1.088577 -0.171018)
+      (xy 1.093611 -0.108354) (xy 1.111963 -0.013373) (xy 1.149047 0.050396) (xy 1.201678 0.096074)
+      (xy 1.24669 0.098497) (xy 1.307597 0.069314) (xy 1.361468 0.007293) (xy 1.375833 -0.089436)
+      (xy 1.382123 -0.172004) (xy 1.412461 -0.205639) (xy 1.474611 -0.211667) (xy 1.58518 -0.23581)
+      (xy 1.647687 -0.303001) (xy 1.658055 -0.358593) (xy 1.626507 -0.426483) (xy 1.546571 -0.476292)
+      (xy 1.448708 -0.493889) (xy 1.391228 -0.514192) (xy 1.375833 -0.579198) (xy 1.36018 -0.69989)
+      (xy 1.310569 -0.762928) (xy 1.249828 -0.776111) (xy 1.165092 -0.744572) (xy 1.109225 -0.660982)
+      (xy 1.093611 -0.566764) (xy 1.074641 -0.510472) (xy 1.006959 -0.493909) (xy 1.003097 -0.493889)
+      (xy 0.887354 -0.474869) (xy 0.805595 -0.425099) (xy 0.776111 -0.358593) (xy 0.330636 -0.358593)
+      (xy 0.314268 -0.375229) (xy 0.612626 -0.661665) (xy 0.792336 -0.823352) (xy 0.944094 -0.932626)
+      (xy 1.079934 -0.995204) (xy 1.211893 -1.016803) (xy 1.337353 -1.005917)) (layer B.SilkS) (width 0.01))
+    (fp_poly (pts (xy -1.246311 -0.983454) (xy -1.10286 -0.917167) (xy -0.943586 -0.801166) (xy -0.787245 -0.659965)
+      (xy -0.490657 -0.375229) (xy -0.765676 -0.096856) (xy -0.88733 0.022176) (xy -1.00084 0.125972)
+      (xy -1.091525 0.201497) (xy -1.135957 0.231869) (xy -1.25626 0.26816) (xy -1.410393 0.278993)
+      (xy -1.566375 0.264347) (xy -1.675695 0.232221) (xy -1.843572 0.124146) (xy -1.96017 -0.018966)
+      (xy -2.026874 -0.185203) (xy -2.045071 -0.362652) (xy -2.044095 -0.368617) (xy -1.799167 -0.368617)
+      (xy -1.77611 -0.308218) (xy -1.743731 -0.267104) (xy -1.679923 -0.239258) (xy -1.56641 -0.220247)
+      (xy -1.423516 -0.210316) (xy -1.271567 -0.209712) (xy -1.130889 -0.218684) (xy -1.021807 -0.237477)
+      (xy -0.973532 -0.257741) (xy -0.925115 -0.333036) (xy -0.922692 -0.390032) (xy -0.930755 -0.427963)
+      (xy -0.950648 -0.453145) (xy -0.995129 -0.468688) (xy -1.076955 -0.4777) (xy -1.20888 -0.483288)
+      (xy -1.317819 -0.486301) (xy -1.517046 -0.487834) (xy -1.655504 -0.478704) (xy -1.742479 -0.456641)
+      (xy -1.787256 -0.419375) (xy -1.799167 -0.368617) (xy -2.044095 -0.368617) (xy -2.016147 -0.539399)
+      (xy -1.941487 -0.703531) (xy -1.822478 -0.843136) (xy -1.660506 -0.946299) (xy -1.533729 -0.987971)
+      (xy -1.385935 -1.005298) (xy -1.246311 -0.983454)) (layer B.SilkS) (width 0.01))
+    (fp_poly (pts (xy 0.158733 -3.590057) (xy 0.355664 -3.577436) (xy 0.436411 -3.566439) (xy 0.862729 -3.457236)
+      (xy 1.269212 -3.284931) (xy 1.649045 -3.055765) (xy 1.99541 -2.775981) (xy 2.301492 -2.45182)
+      (xy 2.560474 -2.089525) (xy 2.765539 -1.695338) (xy 2.900729 -1.309849) (xy 2.940528 -1.110286)
+      (xy 2.967318 -0.864144) (xy 2.980915 -0.591853) (xy 2.981139 -0.313839) (xy 2.967808 -0.050532)
+      (xy 2.940739 0.177641) (xy 2.915049 0.299861) (xy 2.769094 0.722806) (xy 2.564104 1.113563)
+      (xy 2.296621 1.47787) (xy 2.041142 1.748539) (xy 1.734927 2.015845) (xy 1.427769 2.226282)
+      (xy 1.100867 2.39124) (xy 0.79375 2.504102) (xy 0.673142 2.537762) (xy 0.547213 2.561735)
+      (xy 0.398856 2.578013) (xy 0.210963 2.588582) (xy 0.017639 2.594333) (xy -0.185117 2.596538)
+      (xy -0.378105 2.594334) (xy -0.543095 2.588225) (xy -0.661858 2.578713) (xy -0.687917 2.574892)
+      (xy -1.078147 2.473705) (xy -1.466172 2.313218) (xy -1.831677 2.102321) (xy -1.937108 2.028192)
+      (xy -2.298192 1.720713) (xy -2.604449 1.372435) (xy -2.852752 0.988038) (xy -3.039973 0.572199)
+      (xy -3.142674 0.224363) (xy -3.183907 -0.023873) (xy -3.205192 -0.309665) (xy -3.205683 -0.389739)
+      (xy -2.624801 -0.389739) (xy -2.607612 -0.12355) (xy -2.54588 0.10177) (xy -2.432725 0.305012)
+      (xy -2.319782 0.443613) (xy -2.09254 0.644491) (xy -1.839492 0.781823) (xy -1.567336 0.853885)
+      (xy -1.282771 0.858951) (xy -0.992496 0.795299) (xy -0.975894 0.789557) (xy -0.795704 0.699984)
+      (xy -0.593154 0.55266) (xy -0.376145 0.353568) (xy -0.309412 0.284649) (xy -0.213567 0.186451)
+      (xy -0.13489 0.111971) (xy -0.086441 0.073356) (xy -0.079279 0.070555) (xy -0.044733 0.094241)
+      (xy 0.027816 0.158541) (xy 0.127358 0.253314) (xy 0.230133 0.355482) (xy 0.417263 0.534896)
+      (xy 0.579942 0.664274) (xy 0.733756 0.75168) (xy 0.89429 0.805177) (xy 1.07713 0.832825)
+      (xy 1.164166 0.838661) (xy 1.335805 0.842823) (xy 1.465915 0.833128) (xy 1.582753 0.806132)
+      (xy 1.665168 0.777599) (xy 1.900955 0.653153) (xy 2.111106 0.472723) (xy 2.280877 0.250032)
+      (xy 2.331777 0.157101) (xy 2.392217 0.02351) (xy 2.426044 -0.089567) (xy 2.440488 -0.214672)
+      (xy 2.442947 -0.343308) (xy 2.420372 -0.624237) (xy 2.349067 -0.864412) (xy 2.222783 -1.079412)
+      (xy 2.084211 -1.237545) (xy 1.88185 -1.409299) (xy 1.673193 -1.519202) (xy 1.441483 -1.573603)
+      (xy 1.181805 -1.579505) (xy 0.989639 -1.561232) (xy 0.826541 -1.523427) (xy 0.677077 -1.458204)
+      (xy 0.525809 -1.357676) (xy 0.3573 -1.213957) (xy 0.231676 -1.094098) (xy -0.091149 -0.777515)
+      (xy -0.385348 -1.073251) (xy -0.579553 -1.258551) (xy -0.74806 -1.393179) (xy -0.905511 -1.484347)
+      (xy -1.066548 -1.539267) (xy -1.245813 -1.565152) (xy -1.393473 -1.569861) (xy -1.562321 -1.566537)
+      (xy -1.686564 -1.553444) (xy -1.791969 -1.525901) (xy -1.904303 -1.479225) (xy -1.911932 -1.475663)
+      (xy -2.137683 -1.335986) (xy -2.337942 -1.147415) (xy -2.493374 -0.929326) (xy -2.531031 -0.855282)
+      (xy -2.586292 -0.712482) (xy -2.61521 -0.570103) (xy -2.624762 -0.393511) (xy -2.624801 -0.389739)
+      (xy -3.205683 -0.389739) (xy -3.207046 -0.611655) (xy -3.189982 -0.908483) (xy -3.154517 -1.178791)
+      (xy -3.103649 -1.393473) (xy -2.936259 -1.810866) (xy -2.707852 -2.208281) (xy -2.427665 -2.572266)
+      (xy -2.104934 -2.889372) (xy -2.039264 -2.943455) (xy -1.816892 -3.10016) (xy -1.554754 -3.251683)
+      (xy -1.279405 -3.384415) (xy -1.017398 -3.484749) (xy -0.934861 -3.509395) (xy -0.7721 -3.541764)
+      (xy -0.560215 -3.566894) (xy -0.320351 -3.583906) (xy -0.073654 -3.59192) (xy 0.158733 -3.590057)) (layer B.SilkS) (width 0.01))
+  )
+  (module atx:logo3 (layer F.Cu)

Commit message: couronne
Parts:
- added G***: LOGO, atx:couronne3000, F.Cu at (239.2, 113.5)
- added G***: LOGO, atx:couronne1500, F.Cu at (183.1, 162.7)
- added G***: LOGO, atx:couronne1200, F.Cu at (182.8, 151.9)
- added G***: LOGO, atx:couronne10001000, F.Cu at (182.6, 138.2)
- added G***: LOGO, atx:couronne700700, F.Cu at (182.9, 121.5)

Commit message: cc
Parts:
- removed the G*** at (183.1, 162.7)
- removed the G*** at (182.8, 151.9)
- removed the G*** at (182.6, 138.2)
- removed the G*** at (182.9, 121.5)

Commit message: khkhk
Parts:
- added G***: LOGO, atx:3kj, F.Cu at (217.5, 119.0)
- added G***: LOGO, atx:raspi-barre, F.Cu at (181.0, 109.0)
- added G***: LOGO, atx:raspi-barre, F.Cu at (166.0, 109.0)

Commit message: mie a jour esp8266
Parts:
- removed the G*** at (217.5, 119.0)
- removed the G*** at (181.0, 109.0)
- removed the G*** at (166.0, 109.0)
- added G***: LOGO, atx:mort4000, F.Cu at (219.7, 114.2)
- added G***: LOGO, atx:mort4norm, F.Cu at (190.0, 120.7)
- added G***: LOGO, atx:test11, F.Cu at (219.7, 120.2)
- added REF**: PinHeader_1x15_P2.54mm_Vertical, Connector_PinHeader_2.54mm:PinHeader_1x15_P2.54mm_Vertical, F.Cu at (220.0, 189.8)
- added REF**: PinHeader_1x15_P2.54mm_Vertical, Connector_PinHeader_2.54mm:PinHeader_1x15_P2.54mm_Vertical, F.Cu at (220.0, 157.2)
- added REF**: PinHeader_1x15_P2.54mm_Vertical, Connector_PinHeader_2.54mm:PinHeader_1x15_P2.54mm_Vertical, F.Cu at (220.0, 181.0)
- added REF**: PinHeader_1x15_P2.54mm_Vertical, Connector_PinHeader_2.54mm:PinHeader_1x15_P2.54mm_Vertical, F.Cu at (220.0, 183.0)
- added REF**: PinHeader_1x15_P2.54mm_Vertical, Connector_PinHeader_2.54mm:PinHeader_1x15_P2.54mm_Vertical, F.Cu at (220.0, 165.0)
- added REF**: PinHeader_1x15_P2.54mm_Vertical, Connector_PinHeader_2.54mm:PinHeader_1x15_P2.54mm_Vertical, F.Cu at (220.0, 167.0)
- added REF**: PinHeader_1x15_P1.00mm_Vertical, Connector_PinHeader_1.00mm:PinHeader_1x15_P1.00mm_Vertical, F.Cu at (178.0, 173.0)
- added REF**: MountingHole_2.7mm_M2.5_DIN965, MountingHole:MountingHole_2.7mm_M2.5_DIN965, F.Cu at (261.4, 141.3)
- added U2: ESP8266EX-NODEMCU-FRED-chaudier, atx:ESP12F-Devkit-V3-fred-GPIO-1, F.Cu at (239.0, 173.4)
Routing:
- net (no net): track 0.00 -> 4.77 mm
