File: raspberrypi-gpio-40pin.sch (KiCad schematic (older format))
At the start: 15 parts, among them J1 Conn_01x02_Female, J10 Conn_01x02_Female, J2 Conn_01x02_Female, J3 Conn_01x02_Female, J4 Conn_01x02_Female, J5 Conn_01x02_Female, J6 Conn_01x02_Female, J7 Conn_01x02_Female, J8 Conn_01x02_Female, J9 Conn_01x02_Female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

Commit message: mise a jour
Parts:
- added J11, J12, J13, J14, J15, J16, J17, J18, J19, J20, J21, J22, J23, J24, J25, J26, J27, J28, J29, J30: Conn_01x02_Male, atx:PinHeader_1x02_P2.54mm_Vertical, symbol Connector:Conn_01x02_Male
- P1: footprint Connector_PinSocket_2.54mm:PinSocket_2x20_P2.54mm_Vertical -> Connector_PinHeader_2.54mm:PinHeader_2x20_P2.54mm_Vertical
Connections:
- wire segments 76 -> 168
