File: _autosave-raspberrypi-gpio-40pin.kicad_pcb (KiCad board)
At the start: 2 copper layers, 65 x 56 mm, 41 parts, among them J1 Conn_01x02_Female, J10 Conn_01x02_Female, J11 Conn_01x02_Male, J12 Conn_01x02_Male, J13 Conn_01x02_Male, J14 Conn_01x02_Male, J15 Conn_01x02_Male, J16 Conn_01x02_Male, J17 Conn_01x02_Male, J18 Conn_01x02_Male, J19 Conn_01x02_Male, J2 Conn_01x02_Female, J20 Conn_01x02_Male, J21 Conn_01x02_Male, J22 Conn_01x02_Male, J23 Conn_01x02_Male, J24 Conn_01x02_Male, J25 Conn_01x02_Male, J26 Conn_01x02_Male, J27 Conn_01x02_Male, J28 Conn_01x02_Male, J29 Conn_01x02_Male, J3 Conn_01x02_Female, J30 Conn_01x02_Male, J4 Conn_01x02_Female, J5 Conn_01x02_Female, J6 Conn_01x02_Female, J7 Conn_01x02_Female, J8 Conn_01x02_Female, J9 Conn_01x02_Female, P1 Conn_02x20_Odd_Even

Commit message: mie a jour esp8266
Parts:
- removed the G*** at (217.5, 119.0)
- removed the G*** at (181.0, 109.0)
- removed the G*** at (166.0, 109.0)
- added G***: LOGO, atx:mort4000, F.Cu at (219.7, 114.2)
- added G***: LOGO, atx:mort4norm, F.Cu at (190.0, 120.7)
- added G***: LOGO, atx:test11, F.Cu at (219.7, 120.2)
- added REF**: MountingHole_2.7mm, MountingHole:MountingHole_2.7mm, F.Cu at (261.2, 141.2)
- added REF**: PinHeader_1x15_P2.54mm_Vertical_v2, atx:PinHeader_1x15_P2.54mm_Vertical_v2, F.Cu at (220.0, 189.8)
- added REF**: PinHeader_1x15_P2.54mm_Vertical_v2, atx:PinHeader_1x15_P2.54mm_Vertical_v2, F.Cu at (220.0, 157.2)
- added REF**: PinHeader_1x15_P2.54mm_Vertical_v2, atx:PinHeader_1x15_P2.54mm_Vertical_v2, F.Cu at (220.0, 181.0)
- added REF**: PinHeader_1x15_P2.54mm_Vertical_v2, atx:PinHeader_1x15_P2.54mm_Vertical_v2, F.Cu at (220.0, 183.0)
- added REF**: PinHeader_1x15_P2.54mm_Vertical_v2, atx:PinHeader_1x15_P2.54mm_Vertical_v2, F.Cu at (220.0, 165.0)
- added REF**: PinHeader_1x15_P2.54mm_Vertical_v2, atx:PinHeader_1x15_P2.54mm_Vertical_v2, F.Cu at (220.0, 167.0)
- added U2: ESP8266EX-NODEMCU-FRED-chaudier, atx:ESP12F-Devkit-V3-fred-GPIO-1, F.Cu at (239.0, 173.4)
- TR2: value MountingHole_2.7mm_M2.5 -> MountingHole_2.7mm_M2.5 203,3 97,5
- moved TR2 6.60 mm to (196.7, 97.3)
Routing:
- net (no net): track 0.00 -> 282.5 mm
- net +5V: track 115.7 -> 117.3 mm
